File: rfreplacement/rfreplacement.kicad_pcb (KiCad board)
At the start: 2 copper layers, 55.9 x 43.9 mm, 36 parts, among them J1 Conn_01x02, J2 Conn_01x02, J3 Conn_01x02

Commit message: Ver1.2 final. Interactive BOM.
Parts:
- FB3, FB4: value Alternative THT -> 81-BL02RN1R2M2
- LM1117-3.3: value LM1117IMPX-3.3 -> LM1117-3.3
- renumbered THS3716 to THS7316
Changed lines of the file:
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@@
   )
   (paper "A4")
+  (title_block
+    (title "C64 RF Modulator Replacement")
+    (date "2022-03-22")
+    (rev "1.2")
+    (company "For Assy  No.250469")
+  )
   (layers
     (0 "F.Cu" signal)
@@
     (property "Sheetname" "")
     (attr smd)
-    (fp_text reference "THS3716" (at 0 0 90) (layer "F.SilkS")
-      (effects (font (size 0.7 0.7) (thickness 0.15)))
-    )
-    (fp_text value "THS7316" (at 0 3.75) (layer "F.Fab")
-      (effects (font (size 1 1) (thickness 0.15)))
+    (fp_text reference "THS7316" (at 0 0 90) (layer "F.SilkS")
+      (effects (font (size 0.7 0.7) (thickness 0.15)))
+    )
+    (fp_text value "THS7316" (at 0.062 -0.035 90) (layer "F.Fab") hide
+      (effects (font (size 0.7 0.7) (thickness 0.15)))
     )
     (fp_text user "${REFERENCE}" (at 0 0) (layer "F.Fab")
@@
       (effects (font (size 0.7 0.7) (thickness 0.15)))
     )
-    (fp_text value "LM1117IMPX-3.3" (at 0 4.5 90) (layer "F.Fab")
-      (effects (font (size 1 1) (thickness 0.15)))
+    (fp_text value "LM1117-3.3" (at -0.308 -0.056 180) (layer "F.Fab") hide
+      (effects (font (size 0.7 0.7) (thickness 0.15)))
     )
     (fp_text user "${REFERENCE}" (at 0 0) (layer "F.Fab")
@@
       (effects (font (size 0.7 0.7) (thickness 0.15)) (justify mirror))
     )
-    (fp_text value "Alternative THT" (at 3.81 -2.37 -270) (layer "B.Fab")
+    (fp_text value "81-BL02RN1R2M2" (at 3.81 -2.37 -270) (layer "B.Fab")
       (effects (font (size 1 1) (thickness 0.15)) (justify mirror))
     )
@@
       (effects (font (size 0.7 0.7) (thickness 0.15)) (justify mirror))
     )
-    (fp_text value "Alternative THT" (at 3.81 -2.37 -270) (layer "B.Fab")
+    (fp_text value "81-BL02RN1R2M2" (at 3.81 -2.37 -270) (layer "B.Fab")
       (effects (font (size 1 1) (thickness 0.15)) (justify mirror))
     )
