File: rfreplacement/rfreplacement.kicad_sch (KiCad schematic)
At the start: 34 parts, among them J1 Conn_01x02, J2 Conn_01x02, J3 Conn_01x02

Commit message: Ver1.2 final. Interactive BOM.
Parts:
- FB3, FB4: value Alternative THT -> 81-BL02RN1R2M2
- REG2: value LM1117IMPX-3.3 -> LM1117-3.3
Other:
- note added: "FB1, FB2 are alternative SMD equivalents"
- title: RF replacement, analog only -> C64 RF Modulator Replacement
Changed lines of the file:
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@@
 (kicad_sch (version 20211123) (generator eeschema)
-  (paper "A3")
+  (paper "A4")
   (title_block
-    (title "RF replacement, analog only")
-    (date "2019-03-10")
-    (rev "1")
+    (title "C64 RF Modulator Replacement")
+    (date "2022-03-22")
+    (rev "1.2")
     (company "c0pperdragon")
     (comment 1 "github.com/c0pperdragon/A-VideoBoard")
+    (comment 2 "Based on:")
+    (comment 3 "github.com/pmandes/C64-RF-Modulator")
+    (comment 4 "S-Video / Stereo Audio mod:")
   )
   (junction (at 40.64 33.02) (diameter 0) (color 0 0 0 0)
@@
   (wire (pts (xy 106.172 41.656) (xy 104.394 41.656))
     (stroke (width 0) (type default) (color 0 0 0 0))
+  )
+  (text "FB1, FB2 are alternative SMD equivalents" (at 94.234 89.408 0)
+    (effects (font (size 1.524 1.524)) (justify left bottom))
   )
   (label "LUMA_OUT" (at 35.56 66.04 0)
@@
       (effects (font (size 1.524 1.524)))
     )
-    (property "Value" "LM1117IMPX-3.3" (id 1) (at 64.77 182.88 0)
+    (property "Value" "LM1117-3.3" (id 1) (at 64.77 182.88 0)
       (effects (font (size 1.524 1.524)))
     )
@@
     (in_bom yes) (on_board yes)
     (property "Reference" "FB4" (id 0) (at 92.456 80.772 90))
-    (property "Value" "Alternative THT" (id 1) (at 92.456 83.058 90))
+    (property "Value" "81-BL02RN1R2M2" (id 1) (at 92.456 83.058 90))
     (property "Footprint" "Resistor_THT:R_Axial_DIN0207_L6.3mm_D2.5mm_P7.62mm_Horizontal" (id 2) (at 92.456 75.692 90)
       (effects (font (size 1.27 1.27)) hide)
@@
     (in_bom yes) (on_board yes)
     (property "Reference" "FB3" (id 0) (at 92.964 53.086 90))
-    (property "Value" "Alternative THT" (id 1) (at 93.218 54.864 90))
+    (property "Value" "81-BL02RN1R2M2" (id 1) (at 93.218 54.864 90))
     (property "Footprint" "Resistor_THT:R_Axial_DIN0207_L6.3mm_D2.5mm_P7.62mm_Horizontal" (id 2) (at 92.964 55.626 90)
       (effects (font (size 1.27 1.27)) hide)
@@
     )
     (path "/9bf51e3d-f1ce-4052-a53d-f14c0b1c3c61"
-      (reference "FB3") (unit 1) (value "Alternative THT") (footprint "Resistor_THT:R_Axial_DIN0207_L6.3mm_D2.5mm_P7.62mm_Horizontal")
+      (reference "FB3") (unit 1) (value "81-BL02RN1R2M2") (footprint "Resistor_THT:R_Axial_DIN0207_L6.3mm_D2.5mm_P7.62mm_Horizontal")
     )
     (path "/69029636-79e5-47ae-bb14-9bc5dbdeb2b4"
-      (reference "FB4") (unit 1) (value "Alternative THT") (footprint "Resistor_THT:R_Axial_DIN0207_L6.3mm_D2.5mm_P7.62mm_Horizontal")
+      (reference "FB4") (unit 1) (value "81-BL02RN1R2M2") (footprint "Resistor_THT:R_Axial_DIN0207_L6.3mm_D2.5mm_P7.62mm_Horizontal")
     )
     (path "/00000000-0000-0000-0000-00006040665e"
@@
     )
     (path "/00000000-0000-0000-0000-00005c765aab"
-      (reference "REG2") (unit 1) (value "LM1117IMPX-3.3") (footprint "Package_TO_SOT_SMD:SOT-223")
+      (reference "REG2") (unit 1) (value "LM1117-3.3") (footprint "Package_TO_SOT_SMD:SOT-223")
     )
     (path "/00000000-0000-0000-0000-00005c1ae2ca"
